Commit message: changed iiwa model

File: iiwa_agv/urdf/iiwa_agv.gazebo.xacro (robot description, xacro)
@@ -3,4 +3,7 @@
   <gazebo reference="${prefix}agv_link">
     <material>Gazebo/Blue</material>
+  </gazebo>
+  <gazebo reference="${prefix}shengjiangtai">
+    <material>Gazebo/Grey</material>
   </gazebo>
   <gazebo reference="${prefix}base_link">
@@ -27,4 +30,7 @@
   <gazebo reference="${prefix}link_7">
       <material>Gazebo/Yellow</material>
+  </gazebo>
+  <gazebo reference="${prefix}falan">
+      <material>Gazebo/Grey</material>
   </gazebo>
   <gazebo reference="${prefix}pan_link">

File: iiwa_agv/urdf/iiwa_agv.urdf.xacro (robot description, xacro)
@@ -5,4 +5,5 @@
   <xacro:property name="prefix" value="" />
   <xacro:property name="agv_mass" value="50.0" />
+  <xacro:property name="shengjiang_mass" value="10.0" />
   <xacro:property name="xiao_arm_offset_x" value="0.15" />
   <xacro:property name="xiao_arm_offset_y" value="0.5" />
@@ -80,5 +81,5 @@
       <origin xyz="0 0 0" rpy="0 0 0" />
       <geometry>
-        <box size="1 0.5 0.36"/>
+        <box size="1.2 0.7 0.36"/>
       </geometry>
       <material name="blue"/>
@@ -87,7 +88,26 @@
       <origin xyz="0 0 0" rpy="0 0 0" />
       <geometry>
-        <box size="1 0.5 0.36"/>
-      </geometry>
-    </collision>
+        <box size="1.2 0.7 0.36"/>
+      </geometry>
+    </collision>
+  </link>
+  <link name="${prefix}shengjiangtai">
+    <visual>
+      <origin xyz="0 0 0" rpy="0 0 0" />
+      <geometry>
+        <mesh filename="package://iiwa_agv/meshes/shengjiang.STL" />
+      </geometry>
+      <material name="purple"/>
+    </visual>
+    <collision>
+      <origin xyz="0 0 0" rpy="0 0 0" />
+      <geometry>
+        <mesh filename="package://iiwa_agv/meshes/shengjiang.STL" />
+      </geometry>
+    </collision>
+    <inertial>
+      <mass value="${shengjiang_mass}" />
+      <inertia ixx="${shengjiang_mass}" ixy="0.0" ixz="0.0" iyy="${shengjiang_mass}" iyz="0.0" izz="${shengjiang_mass}" />
+    </inertial>
   </link>
   <link name="${prefix}base_link">
@@ -254,4 +274,23 @@
     </xacro:cylinder_inertial>
   </link>
+  <link name="${prefix}falan">
+    <visual>
+      <origin xyz="0 0 0" rpy="0 0 0" />
+      <geometry>
+        <mesh filename="package://iiwa_agv/meshes/falan.STL"/>
+      </geometry>
+      <material name="white"/>
+    </visual>
+    <collision>
+      <origin xyz="0 0 0" rpy="0 0 0" />
+      <geometry>
+        <mesh filename="package://iiwa_agv/meshes/falan.STL"/>
+      </geometry>
+    </collision>
+    <inertial>
+      <mass value="0.1" />
+      <inertia ixx="0.1" ixy="0.0" ixz="0.0" iyy="0.1" iyz="0.0" izz="0.1" />
+    </inertial>
+  </link>
   <link name="${prefix}xiao_arm1_link">
     <visual>
@@ -310,7 +349,12 @@
   <!-- end of link list -->
   <!-- joint list -->
-  <joint name="${prefix}agv_to_base_joint" type="fixed">
-    <origin xyz="0 0 0.18" rpy="0 0 0" />
+  <joint name="${prefix}agv_to_shengjiang" type="fixed">
+    <origin xyz="0.2 0 0.18" rpy="0 0 ${-PI/2.0}" />
     <parent link="${prefix}agv_link" />
+    <child link="${prefix}shengjiangtai" />
+  </joint>
+  <joint name="${prefix}shengjiang_to_base_joint" type="fixed">
+    <origin xyz="0 0.2 0.6" rpy="${-PI/2.0} 0 0" />
+    <parent link="${prefix}shengjiangtai" />
     <child link="${prefix}base_link" />
   </joint>
@@ -370,8 +414,13 @@
     <axis xyz="0 0 0" />
   </joint>
-  <joint name="${prefix}link7_to_pan_joint" type="fixed">
+  <joint name="${prefix}link7_to_falan_joint" type="fixed">
     <parent link="${prefix}link_7" />
+    <child link = "${prefix}falan" />
+    <origin xyz="0.0 0.0 0.126" rpy="${-PI/2.0} 0.0 ${PI/2.0}" />
+  </joint>
+  <joint name="${prefix}falan_to_pan_joint" type="fixed">
+    <parent link="${prefix}falan" />
     <child link = "${prefix}pan_link" />
-    <origin xyz="0.0 0.0 0.126" rpy="0.0 0.0 0.0" />
+    <origin xyz="0.11 0.0 0" rpy="${PI/2.0} 0.0 ${PI/2.0}" />
   </joint>
   <joint name="${prefix}pan_to_xiao_arm1_joint" type="fixed">
