Commit message: add wheels

File: iiwa_agv/urdf/iiwa_agv.urdf.xacro (robot description, xacro)
@@ -92,21 +92,66 @@
     </collision>
   </link>
-  <link name="${prefix}shengjiangtai">
-    <visual>
-      <origin xyz="0 0 0" rpy="0 0 0" />
-      <geometry>
-        <mesh filename="package://iiwa_agv/meshes/shengjiang.STL" />
-      </geometry>
-      <material name="purple"/>
-    </visual>
-    <collision>
-      <origin xyz="0 0 0" rpy="0 0 0" />
-      <geometry>
-        <mesh filename="package://iiwa_agv/meshes/shengjiang.STL" />
-      </geometry>
-    </collision>
-    <inertial>
-      <mass value="${shengjiang_mass}" />
-      <inertia ixx="${shengjiang_mass}" ixy="0.0" ixz="0.0" iyy="${shengjiang_mass}" iyz="0.0" izz="${shengjiang_mass}" />
+  <link name="${prefix}l_f_wheel">
+    <visual>
+       <geometry>
+          <mesh filename="package://iiwa_agv/meshes/wheel.STL" />
+      </geometry>
+    </visual>
+    <collision>
+      <geometry>
+        <mesh filename="package://iiwa_agv/meshes/wheel.STL" />
+      </geometry>
+    </collision>
+    <inertial>
+      <mass value="1" />
+      <inertia ixx="1.0" ixy="0.0" ixz="0.0" iyy="1.0" iyz="0.0" izz="1.0" />
+    </inertial>
+  </link>
+  <link name="${prefix}r_f_wheel">
+    <visual>
+       <geometry>
+          <mesh filename="package://iiwa_agv/meshes/wheel.STL" />
+      </geometry>
+    </visual>
+    <collision>
+      <geometry>
+        <mesh filename="package://iiwa_agv/meshes/wheel.STL" />
+      </geometry>
+    </collision>
+    <inertial>
+      <mass value="1" />
+      <inertia ixx="1.0" ixy="0.0" ixz="0.0" iyy="1.0" iyz="0.0" izz="1.0" />
+    </inertial>
+  </link>
+  <link name="${prefix}l_b_wheel">
+    <visual>
+       <geometry>
+          <mesh filename="package://iiwa_agv/meshes/wheel.STL" />
+      </geometry>
+    </visual>
+    <collision>
+      <geometry>
+        <mesh filename="package://iiwa_agv/meshes/wheel.STL" />
+      </geometry>
+    </collision>
+    <inertial>
+      <mass value="1" />
+      <inertia ixx="1.0" ixy="0.0" ixz="0.0" iyy="1.0" iyz="0.0" izz="1.0" />
+    </inertial>
+  </link>
+  <link name="${prefix}r_b_wheel">
+    <visual>
+       <geometry>
+          <mesh filename="package://iiwa_agv/meshes/wheel.STL" />
+      </geometry>
+    </visual>
+    <collision>
+      <geometry>
+        <mesh filename="package://iiwa_agv/meshes/wheel.STL" />
+      </geometry>
+    </collision>
+    <inertial>
+      <mass value="1" />
+      <inertia ixx="1.0" ixy="0.0" ixz="0.0" iyy="1.0" iyz="0.0" izz="1.0" />
     </inertial>
   </link>
@@ -349,13 +394,28 @@
   <!-- end of link list -->
   <!-- joint list -->
-  <joint name="${prefix}agv_to_shengjiang" type="fixed">
-    <origin xyz="0.2 0 0.18" rpy="0 0 ${-PI/2.0}" />
+  <joint name="${prefix}agv_to_base_joint" type="fixed">
+    <origin xyz="0 0 0.18" rpy="0 0 ${-PI/2.0}" />
     <parent link="${prefix}agv_link" />
-    <child link="${prefix}shengjiangtai" />
-  </joint>
-  <joint name="${prefix}shengjiang_to_base_joint" type="fixed">
-    <origin xyz="0 0.2 0.6" rpy="${-PI/2.0} 0 0" />
-    <parent link="${prefix}shengjiangtai" />
     <child link="${prefix}base_link" />
+  </joint>
+  <joint name="${prefix}agv_to_l_f_wheel" type="fixed">
+    <origin xyz="0.5 0.37 -0.1" rpy="${PI/2.0} ${PI/2.0} 0" />
+    <parent link="${prefix}agv_link" />
+    <child link="${prefix}l_f_wheel" />
+  </joint>
+  <joint name="${prefix}agv_to_r_f_wheel" type="fixed">
+    <origin xyz="-0.5 0.37 -0.1" rpy="${PI/2.0} ${PI/2.0} 0" />
+    <parent link="${prefix}agv_link" />
+    <child link="${prefix}r_f_wheel" />
+  </joint>
+  <joint name="${prefix}agv_to_l_b_wheel" type="fixed">
+    <origin xyz="0.5 -0.37 -0.1" rpy="${PI/2.0} ${PI/2.0} 0" />
+    <parent link="${prefix}agv_link" />
+    <child link="${prefix}l_b_wheel" />
+  </joint>
+  <joint name="${prefix}agv_to_r_b_wheel" type="fixed">
+    <origin xyz="-0.5 -0.37 -0.1" rpy="${PI/2.0} ${PI/2.0} 0" />
+    <parent link="${prefix}agv_link" />
+    <child link="${prefix}r_b_wheel" />
   </joint>
   <joint name="${prefix}joint_a1" type="revolute">

File: parallel_car/urdf/parallel_car.urdf.xacro (robot description, xacro)
@@ -30,5 +30,5 @@
         <visual>
             <geometry>
-                <box size="1 0.5 ${car_height}"/>
+                <box size="1.2 0.7 ${car_height}"/>
      	    </geometry>
             <material name="green"/>
@@ -37,5 +37,5 @@
         <collision>
             <geometry>
-                <box size="1 0.5 0.36"/>
+                <box size="1.2 0.7 0.36"/>
      	    </geometry>
             <origin rpy="0.0 0.0 0.0" xyz="0 0 0.0"/>
@@ -46,4 +46,68 @@
         </inertial>
     </link>
+    <link name="l_f_wheel">
+    <visual>
+       <geometry>
+          <mesh filename="package://parallel_car/meshes/wheel.STL" />
+      </geometry>
+    </visual>
+    <collision>
+      <geometry>
+        <mesh filename="package://parallel_car/meshes/wheel.STL" />
+      </geometry>
+    </collision>
+    <inertial>
+      <mass value="1" />
+      <inertia ixx="1.0" ixy="0.0" ixz="0.0" iyy="1.0" iyz="0.0" izz="1.0" />
+    </inertial>
+  </link>
+  <link name="r_f_wheel">
+    <visual>
+       <geometry>
+          <mesh filename="package://parallel_car/meshes/wheel.STL" />
+      </geometry>
+    </visual>
+    <collision>
+      <geometry>
+        <mesh filename="package://parallel_car/meshes/wheel.STL" />
+      </geometry>
+    </collision>
+    <inertial>
+      <mass value="1" />
+      <inertia ixx="1.0" ixy="0.0" ixz="0.0" iyy="1.0" iyz="0.0" izz="1.0" />
+    </inertial>
+  </link>
+  <link name="l_b_wheel">
+    <visual>
+       <geometry>
+          <mesh filename="package://parallel_car/meshes/wheel.STL" />
+      </geometry>
+    </visual>
+    <collision>
+      <geometry>
+        <mesh filename="package://parallel_car/meshes/wheel.STL" />
+      </geometry>
+    </collision>
+    <inertial>
+      <mass value="1" />
+      <inertia ixx="1.0" ixy="0.0" ixz="0.0" iyy="1.0" iyz="0.0" izz="1.0" />
+    </inertial>
+  </link>
+  <link name="r_b_wheel">
+    <visual>
+       <geometry>
+          <mesh filename="package://parallel_car/meshes/wheel.STL" />
+      </geometry>
+    </visual>
+    <collision>
+      <geometry>
+        <mesh filename="package://parallel_car/meshes/wheel.STL" />
+      </geometry>
+    </collision>
+    <inertial>
+      <mass value="1" />
+      <inertia ixx="1.0" ixy="0.0" ixz="0.0" iyy="1.0" iyz="0.0" izz="1.0" />
+    </inertial>
+  </link>
     <link name="barX_link">
         <inertial>
@@ -298,4 +362,24 @@
         <child link="up_link"/>
     </joint>
+    <joint name="car_to_l_f_wheel" type="fixed">
+    <origin xyz="0.5 0.37 -0.1" rpy="${PI/2.0} ${PI/2.0} 0" />
+    <parent link="car_link" />
+    <child link="l_f_wheel" />
+  </joint>
+  <joint name="car_to_r_f_wheel" type="fixed">
+    <origin xyz="-0.5 0.37 -0.1" rpy="${PI/2.0} ${PI/2.0} 0" />
+    <parent link="car_link" />
+    <child link="r_f_wheel" />
+  </joint>
+  <joint name="car_to_l_b_wheel" type="fixed">
+    <origin xyz="0.5 -0.37 -0.1" rpy="${PI/2.0} ${PI/2.0} 0" />
+    <parent link="car_link" />
+    <child link="l_b_wheel" />
+  </joint>
+  <joint name="agv_to_r_b_wheel" type="fixed">
+    <origin xyz="-0.5 -0.37 -0.1" rpy="${PI/2.0} ${PI/2.0} 0" />
+    <parent link="car_link" />
+    <child link="r_b_wheel" />
+  </joint>
     <!-- spawn the sub links and joints-->
     <xacro:sub_link_joint parent_link="down_link" child_link="down_1" height="${down_height}" radius="${down_radius}" beta="10.0" little_width="${little_width}" little_mass="${little_mass}" />

Commit message: change model

File: iiwa_agv/urdf/iiwa_agv.urdf.xacro (robot description, xacro)
@@ -92,4 +92,23 @@
     </collision>
   </link>
+  <link name="${prefix}control_box">
+    <inertial>
+      <mass value="23" />
+      <inertia ixx="1" ixy="0.0" ixz="0.0" iyy="1" iyz="0.0" izz="1" />
+    </inertial>
+    <visual>
+      <origin xyz="0 0 0" rpy="0 0 0" />
+      <geometry>
+        <box size="0.5 0.483 0.19"/>
+      </geometry>
+      <material name="blue"/>
+    </visual>
+    <collision>
+      <origin xyz="0 0 0" rpy="0 0 0" />
+      <geometry>
+        <box size="0.5 0.483 0.19"/>
+      </geometry>
+    </collision>
+  </link>
   <link name="${prefix}l_f_wheel">
     <visual>
@@ -395,5 +414,5 @@
   <!-- joint list -->
   <joint name="${prefix}agv_to_base_joint" type="fixed">
-    <origin xyz="0 0 0.18" rpy="0 0 ${-PI/2.0}" />
+    <origin xyz="0.2 0 0.18" rpy="0 0 ${-PI/2.0}" />
     <parent link="${prefix}agv_link" />
     <child link="${prefix}base_link" />
@@ -418,4 +437,9 @@
     <parent link="${prefix}agv_link" />
     <child link="${prefix}r_b_wheel" />
+  </joint>
+  <joint name="${prefix}agv_tocontrol_box" type="fixed">
+    <origin xyz="-0.35 0 0.28" rpy="0 0 0" />
+    <parent link="${prefix}agv_link" />
+    <child link="${prefix}control_box" />
   </joint>
   <joint name="${prefix}joint_a1" type="revolute">

File: sim_sys/urdf/sim_sys.urdf.xacro (robot description, xacro)
@@ -2,5 +2,5 @@
 <robot xmlns:xacro="http://wiki.ros.org/xacro">
   <xacro:macro name="sim_sys" params="prefix">
-  <xacro:property name="pi" value="3.1415926535897931" />
+  <xacro:property name="PI" value="3.1415926535897931" />
   <xacro:macro name="cylinder_inertial" params="radius length mass *origin">
     <inertial>
@@ -370,9 +370,28 @@
           <mu2>0.5</mu2>
         </gazebo>
+<link name="${prefix}control_box">
+    <inertial>
+      <mass value="23" />
+      <inertia ixx="1" ixy="0.0" ixz="0.0" iyy="1" iyz="0.0" izz="1" />
+    </inertial>
+    <visual>
+      <origin xyz="0 0 0" rpy="0 0 0" />
+      <geometry>
+        <box size="0.5 0.483 0.19"/>
+      </geometry>
+      <material name="blue"/>
+    </visual>
+    <collision>
+      <origin xyz="0 0 0" rpy="0 0 0" />
+      <geometry>
+        <box size="0.5 0.483 0.19"/>
+      </geometry>
+    </collision>
+  </link>
   <joint
     name="${prefix}agv_iiwa_joint"
     type="fixed">
     <origin
-      xyz="0 0 0.18"
+      xyz="-0.2 0 0.18"
       rpy="0 0 0" />
     <parent
@@ -525,4 +544,9 @@
     <!-- end of link list -->
     <!-- joint list -->
+  <joint name="${prefix}agv_tocontrol_box" type="fixed">
+    <origin xyz="0.35 0 0.28" rpy="0 0 0" />
+    <parent link="${prefix}agv_link" />
+    <child link="${prefix}control_box" />
+  </joint>
     <joint name="${prefix}joint_a1" type="revolute">
       <origin xyz="0 0 0" rpy="0 0 0" />
@@ -580,12 +604,33 @@
       <axis xyz="0 0 0" />
     </joint>
-    <!-- end of joint list -->
-    <joint name="${prefix}pan_joint" type="fixed">
-      <parent link="${prefix}link_7" />
-      <child link = "${prefix}pan_link" />
-      <origin xyz="0.0 0.0 0.12" rpy="1.5708 0.0 0.0" />
-      <axis xyz="0 1 0" />
-      <dynamics damping="0.0" friction="0.0"/>
-    </joint>
+    <link name="${prefix}falan">
+    <visual>
+      <origin xyz="0 0 0" rpy="0 0 0" />
+      <geometry>
+        <mesh filename="package://sim_sys/mesh/falan.STL"/>
+      </geometry>
+      <material name="white"/>
+    </visual>
+    <collision>
+      <origin xyz="0 0 0" rpy="0 0 0" />
+      <geometry>
+        <mesh filename="package://sim_sys/mesh/falan.STL"/>
+      </geometry>
+    </collision>
+    <inertial>
+      <mass value="0.1" />
+      <inertia ixx="0.1" ixy="0.0" ixz="0.0" iyy="0.1" iyz="0.0" izz="0.1" />
+    </inertial>
+  </link>
+  <joint name="${prefix}link7_to_falan_joint" type="fixed">
+    <parent link="${prefix}link_7" />
+    <child link = "${prefix}falan" />
+    <origin xyz="0.0 0.0 0.126" rpy="${-PI/2.0} 0.0 ${PI/2.0}" />
+  </joint>
+    <joint name="${prefix}falan_to_pan_joint" type="fixed">
+    <parent link="${prefix}falan" />
+    <child link = "${prefix}pan_link" />
+    <origin xyz="0.11 0.0 0" rpy="${PI/2.0} 0.0 ${PI/2.0}" />
+  </joint>
     <link name="${prefix}pan_link">
       <visual>
