Commit message: change model and adjust the plan and control part

File: iiwa_agv/urdf/iiwa_agv.urdf.xacro (robot description, xacro)
@@ -53,5 +53,5 @@
     </joint>
     <joint name="${prefix}base_x" type="prismatic">
-        <origin xyz="0.0 0.0 0.18" rpy="0.0 0.0 0.0"/>
+        <origin xyz="0.0 0.0 0.05" rpy="0.0 0.0 0.0"/>
         <parent link="${prefix}virtual_base"/>
         <child link="${prefix}virtual_x"/>
@@ -79,14 +79,14 @@
     </inertial>
     <visual>
-      <origin xyz="0 0 0" rpy="0 0 0" />
-      <geometry>
-        <box size="1.2 0.7 0.36"/>
+      <origin xyz="0 0 0" rpy="${PI/2.0} 0 0" />
+      <geometry>
+        <mesh filename="package://iiwa_agv/meshes/car.STL" />
       </geometry>
       <material name="blue"/>
     </visual>
     <collision>
-      <origin xyz="0 0 0" rpy="0 0 0" />
-      <geometry>
-        <box size="1.2 0.7 0.36"/>
+      <origin xyz="0 0 0" rpy="${PI/2.0} 0 0" />
+      <geometry>
+        <mesh filename="package://iiwa_agv/meshes/car.STL" />
       </geometry>
     </collision>
@@ -111,68 +111,4 @@
     </collision>
   </link>
-  <link name="${prefix}l_f_wheel">
-    <visual>
-       <geometry>
-          <mesh filename="package://iiwa_agv/meshes/wheel.STL" />
-      </geometry>
-    </visual>
-    <collision>
-      <geometry>
-        <mesh filename="package://iiwa_agv/meshes/wheel.STL" />
-      </geometry>
-    </collision>
-    <inertial>
-      <mass value="1" />
-      <inertia ixx="1.0" ixy="0.0" ixz="0.0" iyy="1.0" iyz="0.0" izz="1.0" />
-    </inertial>
-  </link>
-  <link name="${prefix}r_f_wheel">
-    <visual>
-       <geometry>
-          <mesh filename="package://iiwa_agv/meshes/wheel.STL" />
-      </geometry>
-    </visual>
-    <collision>
-      <geometry>
-        <mesh filename="package://iiwa_agv/meshes/wheel.STL" />
-      </geometry>
-    </collision>
-    <inertial>
-      <mass value="1" />
-      <inertia ixx="1.0" ixy="0.0" ixz="0.0" iyy="1.0" iyz="0.0" izz="1.0" />
-    </inertial>
-  </link>
-  <link name="${prefix}l_b_wheel">
-    <visual>
-       <geometry>
-          <mesh filename="package://iiwa_agv/meshes/wheel.STL" />
-      </geometry>
-    </visual>
-    <collision>
-      <geometry>
-        <mesh filename="package://iiwa_agv/meshes/wheel.STL" />
-      </geometry>
-    </collision>
-    <inertial>
-      <mass value="1" />
-      <inertia ixx="1.0" ixy="0.0" ixz="0.0" iyy="1.0" iyz="0.0" izz="1.0" />
-    </inertial>
-  </link>
-  <link name="${prefix}r_b_wheel">
-    <visual>
-       <geometry>
-          <mesh filename="package://iiwa_agv/meshes/wheel.STL" />
-      </geometry>
-    </visual>
-    <collision>
-      <geometry>
-        <mesh filename="package://iiwa_agv/meshes/wheel.STL" />
-      </geometry>
-    </collision>
-    <inertial>
-      <mass value="1" />
-      <inertia ixx="1.0" ixy="0.0" ixz="0.0" iyy="1.0" iyz="0.0" izz="1.0" />
-    </inertial>
-  </link>
   <link name="${prefix}base_link">
     <visual>
@@ -322,5 +258,5 @@
   <link name="${prefix}pan_link">
     <visual>
-      <origin xyz="0 0 0" rpy="${PI/2.0} 0 0" />
+      <origin xyz="0 0 0" rpy="0 0 0" />
       <geometry>
         <mesh filename="package://iiwa_agv/meshes/pan.STL"/>
@@ -329,5 +265,5 @@
     </visual>
     <collision>
-      <origin xyz="0 0 0" rpy="${PI/2.0} 0 0" />
+      <origin xyz="0 0 0" rpy="0 0 0" />
       <geometry>
         <mesh filename="package://iiwa_agv/meshes/pan.STL"/>
@@ -335,5 +271,5 @@
     </collision>
     <xacro:cylinder_inertial radius="0.05" length="0.01" mass="0.01">
-      <origin xyz="0.0 0.0 0.0" rpy="${PI/2.0} 0 0" />
+      <origin xyz="0.0 0.0 0.0" rpy="0 0 0" />
     </xacro:cylinder_inertial>
   </link>
@@ -359,5 +295,5 @@
   <link name="${prefix}xiao_arm1_link">
     <visual>
-      <origin xyz="0 ${xiao_arm_offset_y} 0.02" rpy="${PI/2.0} 0 0" />
+      <origin xyz="0 0 0" rpy="0 0 0" />
       <geometry>
         <mesh filename="package://iiwa_agv/meshes/xiao_arm.STL"/>
@@ -366,5 +302,5 @@
     </visual>
     <collision>
-      <origin xyz="0 ${xiao_arm_offset_y} 0.02" rpy="${PI/2.0} 0 0" />
+      <origin xyz="0 0 0" rpy="0 0 0" />
       <geometry>
         <mesh filename="package://iiwa_agv/meshes/xiao_arm.STL"/>
@@ -377,5 +313,5 @@
   <link name="${prefix}xiao_arm2_link">
     <visual>
-      <origin xyz="${-xiao_arm_offset_x} ${xiao_arm_offset_y} 0.02" rpy="${PI/2.0} 0 0" />
+      <origin xyz="0 0 0" rpy="0 0 0" />
       <geometry>
         <mesh filename="package://iiwa_agv/meshes/xiao_arm.STL"/>
@@ -384,5 +320,5 @@
     </visual>
     <collision>
-      <origin xyz="${-xiao_arm_offset_x} ${xiao_arm_offset_y} 0.02" rpy="${PI/2.0} 0 0" />
+      <origin xyz="0 0 0" rpy="0 0 0" />
       <geometry>
         <mesh filename="package://iiwa_agv/meshes/xiao_arm.STL"/>
@@ -395,5 +331,5 @@
   <link name="${prefix}xiangji_link">
     <visual>
-      <origin xyz="0.0 0.0 0.1" rpy="0 0 0" />
+      <origin xyz="0.0 0.0 0.0" rpy="0 0 0" />
       <geometry>
         <mesh filename="package://iiwa_agv/meshes/xiangji.STL"/>
@@ -414,30 +350,10 @@
   <!-- joint list -->
   <joint name="${prefix}agv_to_base_joint" type="fixed">
-    <origin xyz="0.2 0 0.18" rpy="0 0 ${-PI/2.0}" />
+    <origin xyz="-0.2 0 0.3" rpy="0 0 0" />
     <parent link="${prefix}agv_link" />
     <child link="${prefix}base_link" />
   </joint>
-  <joint name="${prefix}agv_to_l_f_wheel" type="fixed">
-    <origin xyz="0.5 0.37 -0.1" rpy="${PI/2.0} ${PI/2.0} 0" />
-    <parent link="${prefix}agv_link" />
-    <child link="${prefix}l_f_wheel" />
-  </joint>
-  <joint name="${prefix}agv_to_r_f_wheel" type="fixed">
-    <origin xyz="-0.5 0.37 -0.1" rpy="${PI/2.0} ${PI/2.0} 0" />
-    <parent link="${prefix}agv_link" />
-    <child link="${prefix}r_f_wheel" />
-  </joint>
-  <joint name="${prefix}agv_to_l_b_wheel" type="fixed">
-    <origin xyz="0.5 -0.37 -0.1" rpy="${PI/2.0} ${PI/2.0} 0" />
-    <parent link="${prefix}agv_link" />
-    <child link="${prefix}l_b_wheel" />
-  </joint>
-  <joint name="${prefix}agv_to_r_b_wheel" type="fixed">
-    <origin xyz="-0.5 -0.37 -0.1" rpy="${PI/2.0} ${PI/2.0} 0" />
-    <parent link="${prefix}agv_link" />
-    <child link="${prefix}r_b_wheel" />
-  </joint>
   <joint name="${prefix}agv_tocontrol_box" type="fixed">
-    <origin xyz="-0.35 0 0.28" rpy="0 0 0" />
+    <origin xyz="0.35 0 0.41" rpy="0 0 0" />
     <parent link="${prefix}agv_link" />
     <child link="${prefix}control_box" />
@@ -501,25 +417,25 @@
     <parent link="${prefix}link_7" />
     <child link = "${prefix}falan" />
-    <origin xyz="0.0 0.0 0.126" rpy="${-PI/2.0} 0.0 ${PI/2.0}" />
+    <origin xyz="0.0 0.0 0.13" rpy="${-PI/2.0} 0.0 ${PI}" />
   </joint>
   <joint name="${prefix}falan_to_pan_joint" type="fixed">
     <parent link="${prefix}falan" />
     <child link = "${prefix}pan_link" />
-    <origin xyz="0.11 0.0 0" rpy="${PI/2.0} 0.0 ${PI/2.0}" />
+    <origin xyz="0.11 0.0 0" rpy="${PI} 0.0 ${PI/2.0}" />
   </joint>
   <joint name="${prefix}pan_to_xiao_arm1_joint" type="fixed">
     <parent link="${prefix}pan_link" />
     <child link = "${prefix}xiao_arm1_link" />
-    <origin xyz="0.0 0.0 0.0" rpy="0.0 0.0 0.0" />
+    <origin xyz="0.0 0.0 -0.47" rpy="0.0 0.0 0.0" />
   </joint>
   <joint name="${prefix}pan_to_xiao_arm2_joint" type="fixed">
     <parent link="${prefix}pan_link" />
     <child link = "${prefix}xiao_arm2_link" />
-    <origin xyz="0.0 0.0 0.0" rpy="0.0 0.0 0.0" />
+    <origin xyz="-0.15 0.0 -0.47" rpy="0.0 0.0 0.0" />
   </joint>
   <joint name="${prefix}pan_to_xiangji_joint" type="fixed">
     <parent link="${prefix}pan_link" />
     <child link = "${prefix}xiangji_link" />
-    <origin xyz="0.0 0.0 0.0" rpy="0.0 0.0 0.0" />
+    <origin xyz="0.0 0.065 -0.1" rpy="-1.570796 0.0 0.0" />
   </joint>
   <!-- end of joint list -->

File: parallel_car/urdf/parallel_car.urdf.xacro (robot description, xacro)
@@ -30,14 +30,14 @@
         <visual>
             <geometry>
-                <box size="1.2 0.7 ${car_height}"/>
+                <mesh filename="package://parallel_car/meshes/car.STL" />
      	    </geometry>
             <material name="green"/>
-            <origin rpy="0.0 0.0 0.0" xyz="0 0 0.0"/>
-        </visual>
-        <collision>
-            <geometry>
-                <box size="1.2 0.7 0.36"/>
+            <origin rpy="${PI/2.0} 0.0 0.0" xyz="0 0 -0.12"/>
+        </visual>
+        <collision>
+            <geometry>
+                <mesh filename="package://parallel_car/meshes/car.STL" />
      	    </geometry>
-            <origin rpy="0.0 0.0 0.0" xyz="0 0 0.0"/>
+            <origin rpy="${PI/2.0} 0.0 0.0" xyz="0 0 -0.12"/>
         </collision>
         <inertial>
@@ -46,68 +46,4 @@
         </inertial>
     </link>
-    <link name="l_f_wheel">
-    <visual>
-       <geometry>
-          <mesh filename="package://parallel_car/meshes/wheel.STL" />
-      </geometry>
-    </visual>
-    <collision>
-      <geometry>
-        <mesh filename="package://parallel_car/meshes/wheel.STL" />
-      </geometry>
-    </collision>
-    <inertial>
-      <mass value="1" />
-      <inertia ixx="1.0" ixy="0.0" ixz="0.0" iyy="1.0" iyz="0.0" izz="1.0" />
-    </inertial>
-  </link>
-  <link name="r_f_wheel">
-    <visual>
-       <geometry>
-          <mesh filename="package://parallel_car/meshes/wheel.STL" />
-      </geometry>
-    </visual>
-    <collision>
-      <geometry>
-        <mesh filename="package://parallel_car/meshes/wheel.STL" />
-      </geometry>
-    </collision>
-    <inertial>
-      <mass value="1" />
-      <inertia ixx="1.0" ixy="0.0" ixz="0.0" iyy="1.0" iyz="0.0" izz="1.0" />
-    </inertial>
-  </link>
-  <link name="l_b_wheel">
-    <visual>
-       <geometry>
-          <mesh filename="package://parallel_car/meshes/wheel.STL" />
-      </geometry>
-    </visual>
-    <collision>
-      <geometry>
-        <mesh filename="package://parallel_car/meshes/wheel.STL" />
-      </geometry>
-    </collision>
-    <inertial>
-      <mass value="1" />
-      <inertia ixx="1.0" ixy="0.0" ixz="0.0" iyy="1.0" iyz="0.0" izz="1.0" />
-    </inertial>
-  </link>
-  <link name="r_b_wheel">
-    <visual>
-       <geometry>
-          <mesh filename="package://parallel_car/meshes/wheel.STL" />
-      </geometry>
-    </visual>
-    <collision>
-      <geometry>
-        <mesh filename="package://parallel_car/meshes/wheel.STL" />
-      </geometry>
-    </collision>
-    <inertial>
-      <mass value="1" />
-      <inertia ixx="1.0" ixy="0.0" ixz="0.0" iyy="1.0" iyz="0.0" izz="1.0" />
-    </inertial>
-  </link>
     <link name="barX_link">
         <inertial>
@@ -193,10 +129,10 @@
     <link name="wx_visual_link">
         <inertial>
-            <origin xyz="0.03 0.0 0.23" rpy="0.0 0.0 0.0"/>
+            <origin xyz="0.0 0.0 0.0" rpy="${110.0/180.0*PI} 0.0 ${-PI/2.0}"/>
             <mass value="${wx_mass}"/>
             <inertia ixx="${wx_mass}" ixy="0.0" ixz="0.0" iyy="${wx_mass}" iyz="0.0" izz="${wx_mass}"/>
         </inertial>
         <visual>
-            <origin xyz="0.05 0.0 0.25" rpy="${3.0*PI/4.0} 0.0 ${-PI/2.0}"/>
+            <origin xyz="0.0 0.0 0.0" rpy="${110.0/180.0*PI} 0.0 ${-PI/2.0}"/>
             <geometry>
                 <mesh filename="package://parallel_car/meshes/MZ.STL" />
@@ -205,5 +141,5 @@
         </visual>
         <collision>
-            <origin xyz="0.05 0.0 0.25" rpy="0.0 0.0 0.0"/>
+            <origin xyz="0.0 0.0 0.0" rpy="${110.0/180.0*PI} 0.0 ${-PI/2.0}"/>
             <geometry>
                 <mesh filename="package://parallel_car/meshes/MZ.STL" />
@@ -277,19 +213,4 @@
             </geometry>
         </collision>
-    </link>
-    <!-- addon links for support of wx_link -->
-    <link name="addon_Vertical_link">
-        <inertial>
-            <origin xyz="0.0 0.0 ${addon_length/2.0}" rpy="0.0 0.0 0.0"/>
-            <mass value="${little_mass}"/>
-            <inertia ixx="${little_mass}" ixy="0.0" ixz="0.0" iyy="${little_mass}" iyz="0.0" izz="${little_mass}"/>
-        </inertial>
-        <visual>
-            <origin xyz="0.0 0.0 ${addon_length/2.0}" rpy="0.0 0.0 0.0"/>
-            <geometry>
-                <box size="${addon_width} ${addon_width} ${addon_length}"/>
-            </geometry>
-            <material name="purple"/>
-        </visual>
     </link>
     <!-- joints -->
@@ -336,11 +257,11 @@
         <limit lower="${-PI/2.0}" upper="${PI/2.0}" effort="50.0" velocity="2.0"/>
     </joint>
-    <joint name="addon_Vertical_to_wx_visual" type="fixed">
-        <origin xyz="0.0 0.0 ${addon_length}" rpy="0.0 0.0 0.0"/>
-        <parent link="addon_Vertical_link"/>
+    <joint name="littleZ_to_wx_visual" type="fixed">
+        <origin xyz="0.35 0.0 0.25" rpy="0.0 0.0 0.0"/>
+        <parent link="littleZ_link"/>
         <child link="wx_visual_link"/>
     </joint>
     <joint name="wx_visual_to_wx_medium" type="fixed">
-        <origin xyz="0.03 0.0 0.23" rpy="0.0 ${PI/4.0} 0.0"/>
+        <origin xyz="-0.1 0.0 -0.065" rpy="0.0 ${70.0/180.0*PI} 0.0"/>
         <parent link="wx_visual_link"/>
         <child link="wx_medium_link"/>
@@ -362,24 +283,4 @@
         <child link="up_link"/>
     </joint>
-    <joint name="car_to_l_f_wheel" type="fixed">
-    <origin xyz="0.5 0.37 -0.1" rpy="${PI/2.0} ${PI/2.0} 0" />
-    <parent link="car_link" />
-    <child link="l_f_wheel" />
-  </joint>
-  <joint name="car_to_r_f_wheel" type="fixed">
-    <origin xyz="-0.5 0.37 -0.1" rpy="${PI/2.0} ${PI/2.0} 0" />
-    <parent link="car_link" />
-    <child link="r_f_wheel" />
-  </joint>
-  <joint name="car_to_l_b_wheel" type="fixed">
-    <origin xyz="0.5 -0.37 -0.1" rpy="${PI/2.0} ${PI/2.0} 0" />
-    <parent link="car_link" />
-    <child link="l_b_wheel" />
-  </joint>
-  <joint name="agv_to_r_b_wheel" type="fixed">
-    <origin xyz="-0.5 -0.37 -0.1" rpy="${PI/2.0} ${PI/2.0} 0" />
-    <parent link="car_link" />
-    <child link="r_b_wheel" />
-  </joint>
     <!-- spawn the sub links and joints-->
     <xacro:sub_link_joint parent_link="down_link" child_link="down_1" height="${down_height}" radius="${down_radius}" beta="10.0" little_width="${little_width}" little_mass="${little_mass}" />
@@ -395,9 +296,3 @@
     <xacro:sub_link_joint parent_link="up_link" child_link="up_5" height="${up_height}" radius="${up_radius}" beta="290.0" little_width="${little_width}" little_mass="${little_mass}" />
     <xacro:sub_link_joint parent_link="up_link" child_link="up_6" height="${up_height}" radius="${up_radius}" beta="310.0" little_width="${little_width}" little_mass="${little_mass}" />
-    <!--addon joints-->
-    <joint name="littleZ_to_addon_Vertical" type="fixed">
-        <origin xyz="0.0 0.0 0.0" rpy="0.0 0.0 0.0"/>
-        <parent link="littleZ_link"/>
-        <child link="addon_Vertical_link"/>
-    </joint>
 </robot>

File: sim_sys/urdf/sim_sys.urdf.xacro (robot description, xacro)
@@ -23,5 +23,5 @@
                     <mesh filename="package://sim_sys/mesh/MZ.STL" />
                 </geometry>
-                <origin rpy="${pi/2} 0 0" xyz="0 0 0"/>
+                <origin rpy="${pi/2} 0 0" xyz="0.0 0.1 -0.0"/>
             </visual>
             <collision>
@@ -29,5 +29,5 @@
                     <mesh filename="package://sim_sys/mesh/MZ.STL" />
                 </geometry>
-                <origin rpy="${pi/2} 0 0" xyz="0 0 0"/>
+                <origin rpy="${pi/2} 0 0" xyz="0.0 0.1 -0.0"/>
             </collision>
             <xacro:default_inertial mass="10"/>
@@ -51,17 +51,17 @@
       </link>
     <joint name="${prefix}wx_agv2_1" type="revolute">
-            <origin xyz="0.0 0.0 0.0" rpy="-${pi/4} 0.0 0.0"/>
+            <origin xyz="0.0 0.0 0.0" rpy="0 0.0 0"/>
             <parent link="${prefix}wx"/>
             <child link="${prefix}virtual_x_wx"/>
             <axis xyz="1 0 0"/>
-            <limit lower="0" upper="${pi/2}" effort="50" velocity="1.0" />
+            <limit lower="${-pi*2/9}" upper="${pi/9}" effort="50" velocity="1.0" />
       </joint>
       <joint name="${prefix}wx_agv2_2" type="fixed">
-            <origin xyz="0.0 0.0 0.0" rpy="${pi/4} 0.0 0.0"/>
+            <origin xyz="-0.25 0.0 0.0" rpy="0 0 0"/>
             <parent link="${prefix}virtual_x_wx"/>
             <child link="${prefix}virtual_y_wx"/>
       </joint>
       <joint name="${prefix}virtual_agv2" type="fixed">
-            <origin xyz="0.0 0.0 -1.18" rpy="0.0 0.0 0.0"/>
+            <origin xyz="0.0 0.0 -0.96" rpy="0.0 0.0 0.0"/>
             <parent link="${prefix}virtual_y_wx"/>
             <child link="${prefix}agv_link2"/>
@@ -545,5 +545,5 @@
     <!-- joint list -->
   <joint name="${prefix}agv_tocontrol_box" type="fixed">
-    <origin xyz="0.35 0 0.28" rpy="0 0 0" />
+    <origin xyz="-0.35 0 0.28" rpy="0 0 0" />
     <parent link="${prefix}agv_link" />
     <child link="${prefix}control_box" />
@@ -626,10 +626,10 @@
     <parent link="${prefix}link_7" />
     <child link = "${prefix}falan" />
-    <origin xyz="0.0 0.0 0.126" rpy="${-PI/2.0} 0.0 ${PI/2.0}" />
+    <origin xyz="0.0 0.0 0.13" rpy="${-PI/2.0} 0.0 ${PI}" />
   </joint>
     <joint name="${prefix}falan_to_pan_joint" type="fixed">
     <parent link="${prefix}falan" />
     <child link = "${prefix}pan_link" />
-    <origin xyz="0.11 0.0 0" rpy="${PI/2.0} 0.0 ${PI/2.0}" />
+    <origin xyz="0.11 0.0 0" rpy="${PI} 0.0 ${PI/2.0}" />
   </joint>
     <link name="${prefix}pan_link">
