Commit message: add rotation

File: parallel_car/urdf/parallel_car.transmission.xacro (robot description, xacro)
@@ -55,3 +55,12 @@
         </actuator>
     </transmission>
+    <transmission name="rotate_trans">
+        <type>transmission_interface/SimpleTransmission</type>
+        <joint name="littleZ_to_wx_visual">
+            <hardwareInterface>hardware_interface/PositionJointInterface</hardwareInterface>
+        </joint>
+        <actuator name="littleZ_to_wx_visual_motor">
+            <mechanicalReduction>1</mechanicalReduction>
+        </actuator>
+    </transmission>
 </robot>

File: parallel_car/urdf/parallel_car.urdf.xacro (robot description, xacro)
@@ -127,12 +127,19 @@
         </visual>
     </link>
+     <!--link name="connect_link">
+        <inertial>
+            <origin xyz="0.0 0.0 0.0" rpy="0.0 0.0 0.0"/>
+            <mass value="${little_mass}"/>
+            <inertia ixx="${little_mass}" ixy="0.0" ixz="0.0" iyy="${little_mass}" iyz="0.0" izz="${little_mass}"/>
+        </inertial>
+    </link-->
     <link name="wx_visual_link">
         <inertial>
-            <origin xyz="0.0 0.0 0.0" rpy="${110.0/180.0*PI} 0.0 ${-PI/2.0}"/>
+            <origin xyz="0.0 0.0 0.0" rpy="0 0 0"/>
             <mass value="${wx_mass}"/>
             <inertia ixx="${wx_mass}" ixy="0.0" ixz="0.0" iyy="${wx_mass}" iyz="0.0" izz="${wx_mass}"/>
         </inertial>
         <visual>
-            <origin xyz="0.0 0.0 0.0" rpy="${110.0/180.0*PI} 0.0 ${-PI/2.0}"/>
+            <origin xyz="0.0 0.0 0.0" rpy="0 0 0"/>
             <geometry>
                 <mesh filename="package://parallel_car/meshes/MZ.STL" />
@@ -141,5 +148,5 @@
         </visual>
         <collision>
-            <origin xyz="0.0 0.0 0.0" rpy="${110.0/180.0*PI} 0.0 ${-PI/2.0}"/>
+            <origin xyz="0.0 0.0 0.0" rpy="0 0 0"/>
             <geometry>
                 <mesh filename="package://parallel_car/meshes/MZ.STL" />
@@ -172,4 +179,23 @@
             </geometry>
         </visual>
+    </link>
+    <link name="control_box">
+        <inertial>
+            <origin xyz="0.0 0.0 0.0" rpy="0 0 0"/>
+            <mass value="0.5"/>
+            <inertia ixx="0.5" ixy="0.0" ixz="0.0" iyy="0.5" iyz="0.0" izz="0.5"/>
+        </inertial>
+        <visual>
+            <origin xyz="0.0 0.0 0.0" rpy="0 0 0"/>
+            <geometry>
+                <box size="0.5 0.7 0.25"/>
+            </geometry>
+            <material name="grey"/>
+        </visual>
+        <collision>
+            <geometry>
+                <box size="0.5 0.7 0.25"/>
+            </geometry>
+        </collision>
     </link>
     <!-- up and down links -->
@@ -216,5 +242,5 @@
     <!-- joints -->
     <joint name="car_to_barX" type="prismatic">
-        <origin xyz="0.0 0.0 0.18" rpy="0.0 0.0 0.0"/>
+        <origin xyz="0.3 0.0 0.18" rpy="0.0 0.0 0.0"/>
         <parent link="car_link"/>
         <child link="barX_link"/>
@@ -257,9 +283,11 @@
         <limit lower="${-PI/2.0}" upper="${PI/2.0}" effort="50.0" velocity="2.0"/>
     </joint>
-    <joint name="littleZ_to_wx_visual" type="fixed">
-        <origin xyz="0.35 0.0 0.25" rpy="0.0 0.0 0.0"/>
+    <joint name="littleZ_to_wx_visual" type="continuous">
+        <origin xyz="0.5 0.0 0.25" rpy="${110.0/180.0*PI} 0.0 ${-PI/2.0}"/>
         <parent link="littleZ_link"/>
         <child link="wx_visual_link"/>
-    </joint>
+        <axis xyz="0 0 1.0"/>
+    </joint>
+    <!--origin xyz="0.0 0.0 0.0" rpy="${110.0/180.0*PI} 0.0 ${-PI/2.0}"/-->
     <joint name="wx_visual_to_wx_medium" type="fixed">
         <origin xyz="-0.1 0.0 -0.065" rpy="0.0 ${70.0/180.0*PI} 0.0"/>
@@ -274,7 +302,12 @@
     <!-- up and down joints -->
     <joint name="car_to_down" type="fixed">
-        <origin xyz="0.0 0.0 0.18" rpy="0.0 0.0 0.0"/>
+        <origin xyz="0.3 0.0 0.18" rpy="0.0 0.0 0.0"/>
         <parent link="car_link"/>
         <child link="down_link"/>
+    </joint>
+    <joint name="car_to_control_box" type="fixed">
+        <origin xyz="-0.35 0.0 0.3" rpy="0.0 0.0 0.0"/>
+        <parent link="car_link"/>
+        <child link="control_box"/>
     </joint>
     <joint name="littleZ_to_up" type="fixed">

File: sim_sys/urdf/sim_sys.urdf.xacro (robot description, xacro)
@@ -54,14 +54,14 @@
             <parent link="${prefix}wx"/>
             <child link="${prefix}virtual_x_wx"/>
-            <axis xyz="1 0 0"/>
-            <limit lower="${-pi*2/9}" upper="${pi/9}" effort="50" velocity="1.0" />
+            <axis xyz="-1 0 0"/>
+            <limit lower="${-pi/18}" upper="${pi*2/9}" effort="50" velocity="1.0" />
       </joint>
       <joint name="${prefix}wx_agv2_2" type="fixed">
-            <origin xyz="-0.25 0.0 0.0" rpy="0 0 0"/>
+            <origin xyz="0 0.0 0.0" rpy="0 0 0"/>
             <parent link="${prefix}virtual_x_wx"/>
             <child link="${prefix}virtual_y_wx"/>
       </joint>
       <joint name="${prefix}virtual_agv2" type="fixed">
-            <origin xyz="0.0 0.0 -0.96" rpy="0.0 0.0 0.0"/>
+            <origin xyz="0 -0.6 -0.96" rpy="0.0 0.0 0.0"/>
             <parent link="${prefix}virtual_y_wx"/>
             <child link="${prefix}agv_link2"/>
@@ -73,5 +73,5 @@
         </inertial>
         <visual>
-            <origin xyz="0 0 0" rpy="0 0 0" />
+            <origin xyz="0 0 0" rpy="0 0 ${pi/2}" />
             <geometry>
                 <box size="1.2 0.7 0.36"/>
@@ -82,12 +82,12 @@
         </visual>
         <collision>
-            <origin xyz="0 0 0" rpy="0 0 0" />
+            <origin xyz="0 0 0" rpy="0 0 ${pi/2}" />
             <geometry>
-                <box size="1.2 0.7 0.36"/>
+                <box size="1.4 0.9 0.36"/>
             </geometry>
         </collision>
     </link>
     <!-- gazebo -->
-    <gazebo reference="${prefix}agv2_link">
+    <gazebo reference="${prefix}agv_link2">
         <material>Gazebo/DarkGrey</material>
         <mu1>0.5</mu1>
@@ -111,5 +111,5 @@
       </link>
         <joint name="${prefix}lfjoint2" type="fixed">
-            <origin xyz="0.5 0.355 -0.15" rpy="1.5708 1.5708 0.0"/>
+            <origin xyz="0.355 0.5 -0.15" rpy="1.5708 1.5708 0.0"/>
             <parent link="${prefix}agv_link2"/>
             <child link="${prefix}l_f_wheel2"/>
@@ -137,5 +137,5 @@
       </link>
         <joint name="${prefix}rfjoint2" type="fixed">
-            <origin xyz="-0.5 0.355 -0.15" rpy="1.5708 1.5708 0.0"/>
+            <origin xyz="-0.355 0.5 -0.15" rpy="1.5708 1.5708 0.0"/>
             <parent link="${prefix}agv_link2"/>
             <child link="${prefix}r_f_wheel2"/>
@@ -163,5 +163,5 @@
       </link>
         <joint name="${prefix}lbjoint2" type="fixed">
-            <origin xyz="0.5 -0.355 -0.15" rpy="1.5708 1.5708 0.0"/>
+            <origin xyz="0.355 -0.5 -0.15" rpy="1.5708 1.5708 0.0"/>
             <parent link="${prefix}agv_link2"/>
             <child link="${prefix}l_b_wheel2"/>
@@ -189,5 +189,5 @@
       </link>
         <joint name="${prefix}rbjoint2" type="fixed">
-            <origin xyz="-0.5 -0.355 -0.15" rpy="1.5708 1.5708 0.0"/>
+            <origin xyz="-0.355 -0.5 -0.15" rpy="1.5708 1.5708 0.0"/>
             <parent link="${prefix}agv_link2"/>
             <child link="${prefix}r_b_wheel2"/>
@@ -393,5 +393,5 @@
     type="fixed">
     <origin
-      xyz="-0.2 0 0.18"
+      xyz="-0.35 0 0.18"
       rpy="0 0 0" />
     <parent
@@ -545,5 +545,5 @@
     <!-- joint list -->
   <joint name="${prefix}agv_tocontrol_box" type="fixed">
-    <origin xyz="-0.35 0 0.28" rpy="0 0 0" />
+    <origin xyz="0.35 0 0.28" rpy="0 0 0" />
     <parent link="${prefix}agv_link" />
     <child link="${prefix}control_box" />

Commit message: change rotation

File: parallel_car/urdf/parallel_car.transmission.xacro (robot description, xacro)
@@ -57,8 +57,8 @@
     <transmission name="rotate_trans">
         <type>transmission_interface/SimpleTransmission</type>
-        <joint name="littleZ_to_wx_visual">
+        <joint name="rotate_joint">
             <hardwareInterface>hardware_interface/PositionJointInterface</hardwareInterface>
         </joint>
-        <actuator name="littleZ_to_wx_visual_motor">
+        <actuator name="rotate_joint_motor">
             <mechanicalReduction>1</mechanicalReduction>
         </actuator>

File: parallel_car/urdf/parallel_car.urdf.xacro (robot description, xacro)
@@ -136,10 +136,10 @@
     <link name="wx_visual_link">
         <inertial>
-            <origin xyz="0.0 0.0 0.0" rpy="0 0 0"/>
+            <origin xyz="0.0 0.0 0.0" rpy="${110.0/180.0*PI} 0.0 ${-PI/2.0}"/>
             <mass value="${wx_mass}"/>
             <inertia ixx="${wx_mass}" ixy="0.0" ixz="0.0" iyy="${wx_mass}" iyz="0.0" izz="${wx_mass}"/>
         </inertial>
-        <visual>
-            <origin xyz="0.0 0.0 0.0" rpy="0 0 0"/>
+        <!--visual>
+            <origin xyz="0.0 0.0 0.0" rpy="${110.0/180.0*PI} 0.0 ${-PI/2.0}"/>
             <geometry>
                 <mesh filename="package://parallel_car/meshes/MZ.STL" />
@@ -148,5 +148,25 @@
         </visual>
         <collision>
-            <origin xyz="0.0 0.0 0.0" rpy="0 0 0"/>
+            <origin xyz="0.0 0.0 0.0" rpy="${110.0/180.0*PI} 0.0 ${-PI/2.0}"/>
+            <geometry>
+                <mesh filename="package://parallel_car/meshes/MZ.STL" />
+            </geometry>
+        </collision-->
+    </link>
+    <link name="wx_actual_link">
+        <inertial>
+            <origin xyz="0.0 0.0 0.0" rpy="${110.0/180.0*PI} 0.0 ${-PI/2.0}"/>
+            <mass value="${wx_mass}"/>
+            <inertia ixx="${wx_mass}" ixy="0.0" ixz="0.0" iyy="${wx_mass}" iyz="0.0" izz="${wx_mass}"/>
+        </inertial>
+        <visual>
+            <origin xyz="0.0 0.0 0.0" rpy="${110.0/180.0*PI} 0.0 ${-PI/2.0}"/>
+            <geometry>
+                <mesh filename="package://parallel_car/meshes/MZ.STL" />
+            </geometry>
+            <material name="white"/>
+        </visual>
+        <collision>
+            <origin xyz="0.0 0.0 0.0" rpy="${110.0/180.0*PI} 0.0 ${-PI/2.0}"/>
             <geometry>
                 <mesh filename="package://parallel_car/meshes/MZ.STL" />
@@ -283,9 +303,19 @@
         <limit lower="${-PI/2.0}" upper="${PI/2.0}" effort="50.0" velocity="2.0"/>
     </joint>
-    <joint name="littleZ_to_wx_visual" type="continuous">
-        <origin xyz="0.5 0.0 0.25" rpy="${110.0/180.0*PI} 0.0 ${-PI/2.0}"/>
+    <joint name="littleZ_to_wx_visual" type="fixed">
+        <!--origin xyz="0.5 0.0 0.25" rpy="${110.0/180.0*PI} 0.0 ${-PI/2.0}"/-->
+        <origin xyz="0.5 0.0 0.25" rpy="0 0 0"/>
         <parent link="littleZ_link"/>
         <child link="wx_visual_link"/>
-        <axis xyz="0 0 1.0"/>
+        <!--axis xyz="0 0 1.0"/-->
+        <axis xyz="0.5 0 0.18"/>
+    </joint>
+    <joint name="rotate_joint" type="continuous">
+        <!--origin xyz="0.5 0.0 0.25" rpy="${110.0/180.0*PI} 0.0 ${-PI/2.0}"/-->
+        <origin xyz="0 0.0 0" rpy="0 0 0"/>
+        <parent link="wx_visual_link"/>
+        <child link="wx_actual_link"/>
+        <!--axis xyz="0 0 1.0"/-->
+        <axis xyz="0.5 0 0.18"/>
     </joint>
     <!--origin xyz="0.0 0.0 0.0" rpy="${110.0/180.0*PI} 0.0 ${-PI/2.0}"/-->
