Commit message: add second trajectory

File: sim_sys/urdf/sim_sys.urdf.xacro (robot description, xacro)
@@ -55,5 +55,5 @@
             <child link="${prefix}virtual_x_wx"/>
             <axis xyz="1 0 0"/>
-            <limit lower="-${pi/10}" upper="${pi/2}" effort="50" velocity="1.0" />
+            <limit lower="0" upper="${pi/2}" effort="50" velocity="1.0" />
       </joint>
       <joint name="${prefix}wx_agv2_2" type="fixed">
@@ -63,5 +63,5 @@
       </joint>
       <joint name="${prefix}virtual_agv2" type="fixed">
-            <origin xyz="0.0 0.0 -1" rpy="0.0 0.0 0.0"/>
+            <origin xyz="0.0 0.0 -1.18" rpy="0.0 0.0 0.0"/>
             <parent link="${prefix}virtual_y_wx"/>
             <child link="${prefix}agv_link2"/>
@@ -215,5 +215,5 @@
             <child link="${prefix}virtual_x"/>
             <axis xyz="1 0 0"/>
-            <limit lower="-5" upper="5" effort="50" velocity="1.0" />
+            <limit lower="-8" upper="8" effort="50" velocity="1.0" />
       </joint>
       <joint name="${prefix}agv2_viry" type="prismatic">
@@ -222,5 +222,5 @@
             <child link="${prefix}virtual_y"/>
             <axis xyz="0 1 0"/>
-            <limit lower="-5" upper="5" effort="50" velocity="1.0" />
+            <limit lower="-8" upper="8" effort="50" velocity="1.0" />
       </joint>
       <joint name="${prefix}agv2_virz" type="revolute">

Commit message: add fk and get data

File: sim_sys/urdf/sim_sys.urdf.xacro (robot description, xacro)
@@ -719,5 +719,5 @@
       <collision>
         <geometry>
-          <mesh filename="package://sim_sys/mesh/xiao_arm.STL"/>
+          <mesh filename="package://sim_sys/mesh/xiangji.STL"/>
         </geometry>
       </collision>

Commit message: add actual data

File: sim_sys/urdf/sim_sys.urdf.xacro (robot description, xacro)
@@ -63,5 +63,5 @@
       </joint>
       <joint name="${prefix}virtual_agv2" type="fixed">
-            <origin xyz="0 -0.6 -0.96" rpy="0.0 0.0 0.0"/>
+            <origin xyz="0 -0.6 -0.78" rpy="0.0 0.0 0.0"/>
             <parent link="${prefix}virtual_y_wx"/>
             <child link="${prefix}agv_link2"/>
